Commit message: fix urdf file

File: practica1_description/urdf/basic_link.urdf (robot description, URDF)
Before this commit: robot basic_link, 2 links, 1 joints
Joints:
- joint base_link_to_link_1_joint: origin xyz=0 0 0.15 rpy=0 0 0 -> xyz=0.1 0 0.15 rpy=0 0 0

Commit message: added 2nd body and joint

File: practica1_description/urdf/basic_link.urdf (robot description, URDF)
Before this commit: robot basic_link, 2 links, 1 joints
Links:
- added link link_2, mass 1; collision box size=0.1 0.1 0.5; visual box size=0.1 0.1 0.5
- link link_1: mass 1 -> 2
Joints:
- added joint link_1_to_link_2_joint: type revolute, parent link_1, child link_2, origin xyz=0.1 0 0.5 rpy=0 0 0, axis 1 0 0, limit lower=-3.14 upper=3.14 effort=1000.0 velocity=1.0
- joint base_link_to_link_1_joint: limit lower=-1.57 upper=1.57 effort=1000.0 velocity=1.0 -> lower=-1.57 upper=1.57 effort=1000.0 velocity=2.0
