Commit message: Add Point P and scara__simple_controller

File: examen_description/urdf/scara_urdf.xacro (robot description, xacro)
@@ -116,3 +116,10 @@
         <origin xyz="0.5 0 0.1" rpy="0 0 0"/>
     </joint>
+    <link name="P" >
+    </link>
+    <joint name="P_joint" type="fixed">
+        <parent link="link_3"/>
+        <child link="P"/>
+        <origin xyz="0.5 0 0" rpy="0 0 0"/>
+    </joint>
 </robot>

Commit message: fixed dimensions and link positions

File: examen_description/urdf/scara_urdf.xacro (robot description, xacro)
@@ -1,7 +1,14 @@
 <?xml version="1.0" encoding="utf-8"?>
 <robot name="robot_scara" xmlns:xacro="http://ros.org/wiki/xacro">
+    <link name="world">
+    </link>
+    <joint name="world_joint" type="fixed">
+        <parent link="world"/>
+        <child link="base_link"/>
+        <origin xyz="0.0 0 0.0" rpy="0 0 0"/>
+    </joint>
     <link name="base_link">
         <visual>
-            <origin xyz="0.0 0.0 0.0" rpy="0 0 0"/>
+            <origin xyz="0.0 0.0 0.15" rpy="0 0 0"/>
             <geometry>
                 <box size="0.2 0.2 0.3"/>
@@ -12,5 +19,5 @@
         </visual>
         <collision>
-            <origin xyz="0.0 0.0 0.0" rpy="0 0 0"/>
+            <origin xyz="0.0 0.0 0.15" rpy="0 0 0"/>
             <geometry>
                 <box size="0.2 0.2 0.3"/>
@@ -80,7 +87,7 @@
         </visual>
         <collision>
-            <origin xyz="0.05 0.0 0.25" rpy="0.0 0.0 0.0" />
+            <origin xyz="0.25 0.0 0.05" rpy="0.0 0.0 0.0" />
                 <geometry>
-                    <box size="0.25 0.1 0.1" />
+                    <box size="0.5 0.1 0.1" />
                 </geometry>
         </collision>
@@ -98,5 +105,5 @@
         <limit lower="-1.57" upper="1.57" velocity="2.0"
             effort="1000.0"/>
-        <origin xyz="0.1 0 0.15" rpy="0 0 0"/>
+        <origin xyz="0.1 0 0.3" rpy="0 0 0"/>
     </joint>
     <joint name="link_2_joint" type="revolute">
